File: PMOD to BNC Connector/PMOD to BNC Connector.kicad_pcb (KiCad board)
At the start: 2 copper layers, 50 x 85 mm, 14 parts, among them J1 Conn_01x06, J2 Conn_01x06, U1 RH-5000, U2 RH-5000, U3 RH-5000, U4 RH-5000, U5 HL-BNC-KHDA, U6 HL-BNC-KHDA, U7 HL-BNC-KHDA, U8 HL-BNC-KHDA

Commit message: Added Ground Test Points
Parts:
- added U10: RH-5000, Test_point:TEST-TH_BD2.54-P1.4_RED, F.Cu at (147.0, 166.7)
- added U9: RH-5000, Test_point:TEST-TH_BD2.54-P1.4_RED, F.Cu at (147.0, 117.0)
Other:
- board text added: "Property of BYU-Idaho"

Commit message: Fixed 3D models to local project paths
Parts:
- turned U1 to 90 degrees
- turned U10 to 90 degrees
- turned U2 to 90 degrees
- turned U3 to 90 degrees
- turned U4 to 90 degrees
- turned U9 to 90 degrees
Changed lines of the file:
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@@
 	(footprint "Test_point:TEST-TH_BD2.54-P1.4_RED"
 		(layer "F.Cu")
-		(at 147 159.01)
+		(at 147 159.01 90)
 		(property "Reference" "U4"
-			(at 0 -4 0)
+			(at 0 -4 90)
 			(layer "F.SilkS")
 			(hide yes)
@@
 		)
 		(property "Value" "RH-5000"
-			(at 0 4 0)
+			(at 0 4 90)
 			(layer "F.Fab")
 			(hide yes)
@@
 		)
 		(property "Datasheet" ""
-			(at 0 0 0)
+			(at 0 0 90)
 			(layer "F.Fab")
 			(hide yes)
@@
 		)
 		(property "Description" ""
-			(at 0 0 0)
+			(at 0 0 90)
 			(layer "F.Fab")
 			(hide yes)
@@
 		)
 		(property "LCSC Part" "C5277086"
-			(at 0 0 0)
+			(at 0 0 90)
 			(unlocked yes)
 			(layer "F.Fab")
@@
 		)
 		(fp_text user "${REFERENCE}"
-			(at 0 0 0)
+			(at 0 0 90)
 			(layer "F.Fab")
 			(effects
@@
 		)
 		(pad "1" thru_hole circle
-			(at 0 0)
+			(at 0 0 90)
 			(size 1.9 1.9)
 			(drill 1.199998)
@@
 		)
 		(embedded_fonts no)
-		(model "${EASYEDA2KICAD}/easyeda2kicad.3dshapes/TEST-TH_BD2.54-P1.4_RED.wrl"
+		(model "${KIPRJMOD}/Libs/EasyEDA.3dshapes/TEST-TH_BD2.54-P1.4_RED.wrl"
 			(offset
 				(xyz 0 -0 0)
@@
 	(footprint "Test_point:TEST-TH_BD2.54-P1.4_RED"
 		(layer "F.Cu")
-		(at 147 136.15)
+		(at 147 136.15 90)
 		(property "Reference" "U2"
-			(at 0 -4 0)
+			(at 0 -4 90)
 			(layer "F.SilkS")
 			(hide yes)
@@
 		)
 		(property "Value" "RH-5000"
-			(at 0 4 0)
+			(at 0 4 90)
 			(layer "F.Fab")
 			(hide yes)
@@
 		)
 		(property "Datasheet" ""
-			(at 0 0 0)
+			(at 0 0 90)
 			(layer "F.Fab")
 			(hide yes)
@@
 		)
 		(property "Description" ""
-			(at 0 0 0)
+			(at 0 0 90)
 			(layer "F.Fab")
 			(hide yes)
@@
 		)
 		(property "LCSC Part" "C5277086"
-			(at 0 0 0)
+			(at 0 0 90)
 			(unlocked yes)
 			(layer "F.Fab")
@@
 		)
 		(fp_text user "${REFERENCE}"
-			(at 0 0 0)
+			(at 0 0 90)
 			(layer "F.Fab")
 			(effects
@@
 		)
 		(pad "1" thru_hole circle
-			(at 0 0)
+			(at 0 0 90)
 			(size 1.9 1.9)
 			(drill 1.199998)
@@
 		)
 		(embedded_fonts no)
-		(model "${EASYEDA2KICAD}/easyeda2kicad.3dshapes/TEST-TH_BD2.54-P1.4_RED.wrl"
+		(model "${KIPRJMOD}/Libs/EasyEDA.3dshapes/TEST-TH_BD2.54-P1.4_RED.wrl"
 			(offset
 				(xyz 0 -0 0)
@@
 	(footprint "Test_point:TEST-TH_BD2.54-P1.4_RED"
 		(layer "F.Cu")
-		(at 147 147.58)
+		(at 147 147.58 90)
 		(property "Reference" "U3"
-			(at 0 -4 0)
+			(at 0 -4 90)
 			(layer "F.SilkS")
 			(hide yes)
@@
 		)
 		(property "Value" "RH-5000"
-			(at 0 4 0)
+			(at 0 4 90)
 			(layer "F.Fab")
 			(hide yes)
@@
 		)
 		(property "Datasheet" ""
-			(at 0 0 0)
+			(at 0 0 90)
 			(layer "F.Fab")
 			(hide yes)
@@
 		)
 		(property "Description" ""
-			(at 0 0 0)
+			(at 0 0 90)
 			(layer "F.Fab")
 			(hide yes)
@@
 		)
 		(property "LCSC Part" "C5277086"
-			(at 0 0 0)
+			(at 0 0 90)
 			(unlocked yes)
 			(layer "F.Fab")
@@
 		)
 		(fp_text user "${REFERENCE}"
-			(at 0 0 0)
+			(at 0 0 90)
 			(layer "F.Fab")
 			(effects
@@
 		)
 		(pad "1" thru_hole circle
-			(at 0 0)
+			(at 0 0 90)
 			(size 1.9 1.9)
 			(drill 1.199998)
@@
 		)
 		(embedded_fonts no)
-		(model "${EASYEDA2KICAD}/easyeda2kicad.3dshapes/TEST-TH_BD2.54-P1.4_RED.wrl"
+		(model "${KIPRJMOD}/Libs/EasyEDA.3dshapes/TEST-TH_BD2.54-P1.4_RED.wrl"
 			(offset
 				(xyz 0 -0 0)
@@
 	(footprint "Test_point:TEST-TH_BD2.54-P1.4_RED"
 		(layer "F.Cu")
-		(at 147 124.72)
+		(at 147 124.72 90)
 		(property "Reference" "U1"
-			(at 0 -4 0)
+			(at 0 -4 90)
 			(layer "F.SilkS")
 			(hide yes)
@@
 		)
 		(property "Value" "RH-5000"
-			(at 0 4 0)
+			(at 0 4 90)
 			(layer "F.Fab")
 			(hide yes)
@@
 		)
 		(property "Datasheet" ""
-			(at 0 0 0)
+			(at 0 0 90)
 			(layer "F.Fab")
 			(hide yes)
@@
 		)
 		(property "Description" ""
-			(at 0 0 0)
+			(at 0 0 90)
 			(layer "F.Fab")
 			(hide yes)
@@
 		)
 		(property "LCSC Part" "C5277086"
-			(at 0 0 0)
+			(at 0 0 90)
 			(unlocked yes)
 			(layer "F.Fab")
@@
 		)
 		(fp_text user "${REFERENCE}"
-			(at 0 0 0)
+			(at 0 0 90)
 			(layer "F.Fab")
 			(effects
@@
 		)
 		(pad "1" thru_hole circle
-			(at 0 0)
+			(at 0 0 90)
 			(size 1.9 1.9)
 			(drill 1.199998)
@@
 		)
 		(embedded_fonts no)
-		(model "${EASYEDA2KICAD}/easyeda2kicad.3dshapes/TEST-TH_BD2.54-P1.4_RED.wrl"
+		(model "${KIPRJMOD}/Libs/EasyEDA.3dshapes/TEST-TH_BD2.54-P1.4_RED.wrl"
 			(offset
 				(xyz 0 -0 0)
@@
 	(footprint "Test_point:TEST-TH_BD2.54-P1.4_RED"
 		(layer "F.Cu")
-		(at 147 117)
+		(at 147 117 90)
 		(property "Reference" "U9"
-			(at 0 -4 0)
+			(at 0 -4 90)
 			(layer "F.SilkS")
 			(hide yes)
@@
 		)
 		(property "Value" "RH-5000"
-			(at 0 4 0)
+			(at 0 4 90)
 			(layer "F.Fab")
 			(hide yes)
@@
 		)
 		(property "Datasheet" ""
-			(at 0 0 0)
+			(at 0 0 90)
 			(layer "F.Fab")
 			(hide yes)
@@
 		)
 		(property "Description" ""
-			(at 0 0 0)
+			(at 0 0 90)
 			(layer "F.Fab")
 			(hide yes)
@@
 		)
 		(property "LCSC Part" "C5277086"
-			(at 0 0 0)
+			(at 0 0 90)
 			(unlocked yes)
 			(layer "F.Fab")
@@
 		)
 		(pad "1" thru_hole circle
-			(at 0 0)
+			(at 0 0 90)
 			(size 1.9 1.9)
 			(drill 1.199998)
@@
 		)
 		(embedded_fonts no)
-		(model "${EASYEDA2KICAD}/easyeda2kicad.3dshapes/TEST-TH_BD2.54-P1.4_RED.wrl"
+		(model "${KIPRJMOD}/Libs/EasyEDA.3dshapes/TEST-TH_BD2.54-P1.4_RED.wrl"
 			(offset
 				(xyz 0 -0 0)
@@
 	(footprint "Test_point:TEST-TH_BD2.54-P1.4_RED"
 		(layer "F.Cu")
-		(at 147 166.73)
+		(at 147 166.73 90)
 		(property "Reference" "U10"
-			(at 0 -4 0)
+			(at 0 -4 90)
 			(layer "F.SilkS")
 			(hide yes)
@@
 		)
 		(property "Value" "RH-5000"
-			(at 0 4 0)
+			(at 0 4 90)
 			(layer "F.Fab")
 			(hide yes)
@@
 		)
 		(property "Datasheet" ""
-			(at 0 0 0)
+			(at 0 0 90)
 			(layer "F.Fab")
 			(hide yes)
@@
 		)
 		(property "Description" ""
-			(at 0 0 0)
+			(at 0 0 90)
 			(layer "F.Fab")
 			(hide yes)
@@
 		)
 		(property "LCSC Part" "C5277086"
-			(at 0 0 0)
+			(at 0 0 90)
 			(unlocked yes)
 			(layer "F.Fab")
@@
 		)
 		(fp_text user "${REFERENCE}"
-			(at 0 0 0)
+			(at 0 0 90)
 			(layer "F.Fab")
 			(effects
@@
 		)
 		(pad "1" thru_hole circle
-			(at 0 0)
+			(at 0 0 90)
 			(size 1.9 1.9)
 			(drill 1.199998)
@@
 		)
 		(embedded_fonts no)
-		(model "${EASYEDA2KICAD}/easyeda2kicad.3dshapes/TEST-TH_BD2.54-P1.4_RED.wrl"
+		(model "${KIPRJMOD}/Libs/EasyEDA.3dshapes/TEST-TH_BD2.54-P1.4_RED.wrl"
 			(offset
 				(xyz 0 -0 0)
@@
 		)
 		(embedded_fonts no)
-		(model "C:/Users/Jacob Deschamps/Documents/KiCad/Projects/PMOD to BNC Connector/Libs/EasyEDA.3dshapes/BNC-TH_L12.0-W12.0.wrl"
+		(model "${KIPRJMOD}/Libs/EasyEDA.3dshapes/BNC-TH_L12.0-W12.0.wrl"
 			(offset
 				(xyz 0 -0 0)
