File: PMOD to BNC Connector/PMOD to BNC Connector.kicad_sch (KiCad schematic)
At the start: 14 parts, among them J1 Conn_01x06, J2 Conn_01x06, U1 RH-5000, U2 RH-5000, U3 RH-5000, U4 RH-5000, U5 HL-BNC-KHDA, U6 HL-BNC-KHDA, U7 HL-BNC-KHDA, U8 HL-BNC-KHDA

Commit message: Added Ground Test Points
Parts:
- added U10, U9: RH-5000, Test_point:TEST-TH_BD2.54-P1.4_RED, symbol Test_point:RH-5000
Connections:
- net GND: now also U10.1, U9.1
Changed lines of the file:
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@@
+	)
+	(junction
+		(at 62.23 113.03)
+		(diameter 0)
+		(color 0 0 0 0)
 	)
 	(junction
@@
 	)
 	(junction
+		(at 62.23 45.72)
+		(diameter 0)
+		(color 0 0 0 0)
+	)
+	(junction
 		(at 80.01 33.02)
 		(diameter 0)
@@
 	(wire
 		(pts
+			(xy 41.91 113.03) (xy 62.23 113.03)
+		)
+		(stroke
+			(width 0)
+			(type default)
+		)
+	)
+	(wire
+		(pts
 			(xy 73.66 62.23) (xy 73.66 77.47)
 		)
@@
 	(wire
 		(pts
+			(xy 40.64 45.72) (xy 62.23 45.72)
+		)
+		(stroke
+			(width 0)
+			(type default)
+		)
+	)
+	(wire
+		(pts
 			(xy 74.93 21.59) (xy 74.93 40.64)
 		)
@@
 	(wire
 		(pts
-			(xy 62.23 106.68) (xy 62.23 116.84)
+			(xy 62.23 106.68) (xy 62.23 113.03)
 		)
 		(stroke
@@
 	(wire
 		(pts
+			(xy 62.23 45.72) (xy 62.23 52.07)
+		)
+		(stroke
+			(width 0)
+			(type default)
+		)
+	)
+	(wire
+		(pts
 			(xy 62.23 52.07) (xy 62.23 54.61)
 		)
@@
 	(wire
 		(pts
-			(xy 62.23 40.64) (xy 62.23 52.07)
+			(xy 62.23 40.64) (xy 62.23 45.72)
 		)
 		(stroke
@@
 		(pts
 			(xy 93.98 114.3) (xy 111.76 114.3)
+		)
+		(stroke
+			(width 0)
+			(type default)
+		)
+	)
+	(wire
+		(pts
+			(xy 62.23 113.03) (xy 62.23 116.84)
 		)
 		(stroke
@@
 	)
 	(symbol
+		(lib_id "Test_point:RH-5000")
+		(at 36.83 113.03 0)
+		(unit 1)
+		(exclude_from_sim no)
+		(in_bom yes)
+		(on_board yes)
+		(dnp no)
+		(fields_autoplaced yes)
+		(property "Reference" "U9"
+			(at 34.29 105.41 0)
+			(effects
+				(font
+					(size 1.27 1.27)
+				)
+			)
+		)
+		(property "Value" "RH-5000"
+			(at 34.29 107.95 0)
+			(effects
+				(font
+					(size 1.27 1.27)
+				)
+			)
+		)
+		(property "Footprint" "Test_point:TEST-TH_BD2.54-P1.4_RED"
+			(at 36.83 120.65 0)
+			(effects
+				(font
+					(size 1.27 1.27)
+				)
+				(hide yes)
+			)
+		)
+		(property "Datasheet" ""
+			(at 36.83 113.03 0)
+			(effects
+				(font
+					(size 1.27 1.27)
+				)
+				(hide yes)
+			)
+		)
+		(property "Description" ""
+			(at 36.83 113.03 0)
+			(effects
+				(font
+					(size 1.27 1.27)
+				)
+				(hide yes)
+			)
+		)
+		(property "LCSC Part" "C5277086"
+			(at 36.83 123.19 0)
+			(effects
+				(font
+					(size 1.27 1.27)
+				)
+				(hide yes)
+			)
+		)
+		(pin "1"
+		)
+		(instances
+			(project "PMOD to BNC Connector"
+				(path "/c78f13c0-c6c4-40d5-87d9-3ba336170ebc"
+					(reference "U9")
+					(unit 1)
+				)
+			)
+		)
+	)
+	(symbol
 		(lib_id "EasyEDA:HL-BNC-KHDA")
 		(at 57.15 33.02 0)
@@
 					(unit 1)
 				)
+			)
+		)
+	)
+	(symbol
+		(lib_id "Test_point:RH-5000")
+		(at 35.56 45.72 0)
+		(unit 1)
+		(exclude_from_sim no)
+		(in_bom yes)
+		(on_board yes)
+		(dnp no)
+		(fields_autoplaced yes)
+		(property "Reference" "U10"
+			(at 33.02 38.1 0)
+			(effects
+				(font
+					(size 1.27 1.27)
+				)
+			)
+		)
+		(property "Value" "RH-5000"
+			(at 33.02 40.64 0)
+			(effects
+				(font
+					(size 1.27 1.27)
+				)
+			)
+		)
+		(property "Footprint" "Test_point:TEST-TH_BD2.54-P1.4_RED"
+			(at 35.56 53.34 0)
+			(effects
+				(font
+					(size 1.27 1.27)
+				)
+				(hide yes)
+			)
+		)
+		(property "Datasheet" ""
+			(at 35.56 45.72 0)
+			(effects
+				(font
+					(size 1.27 1.27)
+				)
+				(hide yes)
+			)
+		)
+		(property "Description" ""
+			(at 35.56 45.72 0)
+			(effects
+				(font
+					(size 1.27 1.27)
+				)
+				(hide yes)
+			)
+		)
+		(property "LCSC Part" "C5277086"
+			(at 35.56 55.88 0)
+			(effects
+				(font
+					(size 1.27 1.27)
+				)
+				(hide yes)
+			)
+		)
+		(pin "1"
+		)
+		(instances
+			(project "PMOD to BNC Connector"
+				(path "/c78f13c0-c6c4-40d5-87d9-3ba336170ebc"
+					(reference "U10")
+					(unit 1)
+				)

Commit message: V2 Complete
Parts:
- added H1, H2: MountingHole, MountingHole:MountingHole_3.5mm, symbol Mechanical:MountingHole
- added U11, U12: RH-5000, CONN1_1514-2_KEY, symbol New_test_point:1514-2
- U1, U10, U2, U3, U4, U9: footprint Test_point:TEST-TH_BD2.54-P1.4_RED -> CONN1_1514-2_KEY; symbol Test_point:RH-5000 -> New_test_point:1514-2; Height (none) -> 7.14; Manufacturer_Name (none) -> Keystone Electronics; Manufacturer_Part_Number (none) -> 1514-2; Mouser Part Number (none) -> 534-1514-2; Mouser Price/Stock (none) -> https://www.mouser.co.uk/ProductDetail/Keystone-Electronics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
Connections:
- net GND: now also U11.1, U12.1

Commit message: Small tweaks
Parts:
- J1: now left out of the parts list
Changed lines of the file:
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@@
 		(unit 1)
 		(exclude_from_sim no)
-		(in_bom yes)
+		(in_bom no)
 		(on_board yes)
 		(dnp no)
